File: BF_FluidNC/BF_FluidNC.kicad_pcb (KiCad board)
At the start: 2 copper layers, 80.5 x 43.2 mm, 16 parts, among them J1 Conn_01x03_Socket, J2 Conn_Stepper, J3 Conn_Stepper, J4 Conn_Stepper, J5 Barrel_Jack_MountingPin, U1 ESP32-WROOM-32D, U2 A4988_STEPPER_MOTOR_DRIVER_CA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, U3 A4988_STEPPER_MOTOR_DRIVER_CA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, U4 A4988_STEPPER_MOTOR_DRIVER_CA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

Commit message: updated PCB from review notes
Parts:
- U1: footprint ESP32-WROOM-32D:ESP32-WROOMD-Devboard -> ESP32-WROOM-32D:ESP32-WROOMD-Devboard_Truncated
Routing:
- net Net-(J2-B-): track 24.7 -> 21.7 mm
- net Net-(J3-B+): track 12.9 -> 15.3 mm
- net +3V3: track 215.5 -> 217.6 mm
- net +12V: track 121.2 -> 123.1 mm
- net Net-(J3-A+): track 17.0 -> 18.5 mm
- net Net-(J2-B+): track 16.6 -> 15.4 mm
- net PWMOUT: track 25.5 -> 24.5 mm
- net Net-(J3-A-): track 18.5 -> 19.3 mm
- net Net-(J4-A+): track 18.8 -> 19.6 mm

Commit message: new gerbers
Parts:
- added G***: LOGO, LOGO, B.Cu at (141.0, 87.5)
- added G***: LOGO, LOGO, B.Cu at (187.5, 88.5)
- moved G*** 1.00 mm to (132.2, 74.5)
Routing:
- net +3V3: track 217.6 -> 214.3 mm
- net Net-(U4-~{RESET}): track 0.00 -> 2.54 mm
- net Net-(U3-~{RESET}): track 0.00 -> 2.54 mm
- net Net-(U2-~{RESET}): track 0.00 -> 2.54 mm
- net Net-(J2-A+): track 17.2 -> 18.1 mm
- net Net-(J2-B+): track 15.4 -> 16.1 mm
Other:
- board text added: "3V3 40mA"
- board text added: "A4988"
